File: chip8-pcb/chip8-pcb.kicad_sch (KiCad schematic)
At the start: 2 parts, among them J1 Header, J2 Header

Commit message: chip8-pcb: final v1 version
Parts:
- removed J1, J2: Header, symbol Connector:Conn_01x09_Socket
- added BZ1: MLT-8540, chip8-pcb:MLT-8540, symbol chip8-pcb:Buzzer_4P
- added C1: 10u, Capacitor_SMD:C_0603_1608Metric, symbol Device:C_Small
- added C2, C3, C9: 100n, Capacitor_SMD:C_0603_1608Metric, symbol Device:C_Small
- added C4, C5: 22u, Capacitor_SMD:C_0603_1608Metric, symbol Device:C_Small
- added C6: 47u, Capacitor_SMD:CP_Elec_6.3x5.4, symbol Device:C_Polarized_Small
- added C7, C8: 1u, Capacitor_SMD:C_0603_1608Metric, symbol Device:C_Small
- added D1: RED, LED_SMD:LED_0805_2012Metric, symbol Device:LED_Small_Filled
- added D2: GREEN, LED_SMD:LED_0805_2012Metric, symbol Device:LED_Small_Filled
- added D3: SS32, Diode_SMD:D_SMA, symbol Device:D_Schottky_Small_Filled
- added F1: 1A, Fuse:Fuse_0603_1608Metric, symbol Device:Fuse_Small
- added H1, H10, H11, H12, H2, H3, H4, H9: ~, MountingHole:MountingHole_2.7mm_M2.5, symbol Mechanical:MountingHole
- added H5, H6, H7, H8: ~, MountingHole:MountingHole_2.2mm_M2, symbol Mechanical:MountingHole
- added J3: Battery, chip8-pcb:BOOMELE_PH-2P_1x2P_P2.00mm_Horizontal, symbol Connector_Generic_MountingPin:Conn_01x02_MountingPin
- added J4: Matrix Keypad, chip8-pcb:AZDelivery_Keypad_4x4_Matrix_P2.54mm, symbol chip8-pcb:Keypad_4x4
- added J5: Display, Connector_PinHeader_2.54mm:PinHeader_1x07_P2.54mm_Horizontal, symbol Connector_Generic:Conn_01x07
- added JP1, JP3, JP4: ~, Jumper:SolderJumper-2_P1.3mm_Open_RoundedPad1.0x1.5mm, symbol Jumper:SolderJumper_2_Open
- added JP2: ~, Jumper:SolderJumper-2_P1.3mm_Open_RoundedPad1.0x1.5mm, symbol Jumper:Jumper_2_Small_Open
- added L1: 10u, Inductor_SMD:L_Sunlord_SWPA4030S, symbol Device:L_Small
- added Q1: S8050, Package_TO_SOT_SMD:SOT-23, symbol Transistor_BJT:MMBT2222A
- added Q2: BCM857BS, Package_TO_SOT_SMD:SOT-363_SC-70-6, symbol Device:Q_Dual_PNP_PNP_E1B1C2E2B2C1
- added Q3: CJ2301, Package_TO_SOT_SMD:SOT-23, symbol Device:Q_PMOS_GSD
- added R1, R14: 1k, Resistor_SMD:R_0603_1608Metric, symbol Device:R_Small
- added R10, R11, R17, R18, R19, R20, R21, R22, R23, R4, R5, R6, R7, R8, R9: 22, Resistor_SMD:R_0603_1608Metric, symbol Device:R_Small
- added R12: 470, Resistor_SMD:R_0603_1608Metric, symbol Device:R_Small
- added R13: 0, Resistor_SMD:R_0603_1608Metric, symbol Device:R_Small
- added R15: 10k, Resistor_SMD:R_0603_1608Metric, symbol Device:R_Small
- added R16: 47k, Resistor_SMD:R_0603_1608Metric, symbol Device:R_Small
- added R2, R3: 1.2k, Resistor_SMD:R_0603_1608Metric, symbol Device:R_Small
- added SW1: SHDN, Button_Switch_SMD:SW_SPDT_CK_JS102011SAQN, symbol Switch:SW_SPDT
- added U1: TP5400, Package_SO:HTSOP-8-1EP_3.9x4.9mm_P1.27mm_EP2.4x3.2mm_ThermalVias, symbol chip8-pcb:TP5400
- added U2: AP2112K-3.3, Package_TO_SOT_SMD:SOT-23-5, symbol Regulator_Linear:AP2112K-3.3
- added U3: W25Q128JVS, Package_SO:SOIC-8_5.23x5.23mm_P1.27mm, symbol Memory_Flash:W25Q128JVS
- added U4: ESP32-C3-ZERO, chip8-pcb:WaveShare_ESP32-C3-ZERO, symbol chip8-pcb:ESP32-C3-ZERO
Connections:
- new net: JP1.2 (B), R2.1, R3.2
- new net: SW1.2 (B), U2.3 (EN)
- new net: C1.1, F1.1, R1.1, U1.5 (VCC)
- new net: D1.2 (A), D2.2 (A), R1.2
- new net: Q2.3 (C2), Q3.1 (G), R16.1
- new net: BZ1.1 (+), R13.2, R14.1
- new net: BZ1.2 (-), Q1.3 (C), R14.2
- new net: D3.2 (A), L1.1, U1.8 (LX)
- new net: R7.1, U4.15 (GP18)
- new net: J4.5 (R4), R7.2
- new net: R20.2, U4.7 (GP3)
- new net: R17.2, U4.5 (GP1)
- new net: R2.2, U1.3 (PROG)
- new net: D1.1 (K), U1.2 (~{CHRG})
- new net: D2.1 (K), U1.4 (~{STDBY})
- new net: R11.1, U4.11 (GP7)
- new net: J4.9 (C4), R11.2
- new net: R12.1, U4.10 (GP6)
- new net: R10.1, U4.12 (GP8)
- new net: R9.1, U4.13 (GP9)
- new net: R8.1, U4.14 (GP10)
- new net: R6.1, U4.16 (GP19)
- new net: R4.1, U4.17 (GP20)
- new net: R5.1, U4.18 (GP21)
- new net: R18.2, U4.4 (GP0)
- new net: R19.2, U4.6 (GP2)
- new net: R21.2, U4.8 (GP4)
- new net: R22.2, U4.9 (GP5)
- new net: JP4.2 (B), U3.3 (IO2)
- new net: Q1.1 (B), R12.2
- new net: J4.3 (R2), R4.2
- new net: J4.2 (R1), R5.2
- new net: J4.4 (R3), R6.2
- new net: J4.6 (C1), R8.2
- new net: J4.7 (C2), R9.2
- new net: J4.8 (C3), R10.2
- new net: JP3.2 (B), U3.7 (IO3)
- new net: Q2.2 (B1), Q2.5 (B2), Q2.6 (C1), R15.1
- new net +3.3V: C8.1, C9.1, J5.7 (Pin_7), R13.1, R23.2, U2.5 (VOUT), U3.8 (VCC), U4.3 (3V3)
- new net +5V: C3.1, C6.1, C7.1, D3.1 (K), Q2.4 (E2), Q3.2 (S), SW1.1 (A), U1.1 (VOUT), U2.1 (VIN)
- new net +BATT: C2.1, C4.1, C5.1, J3.2 (Pin_2), JP2.1 (A), L1.2, U1.6 (BAT)
- new net GND: C1.2, C2.2, C3.2, C4.2, C5.2, C6.2, C7.2, C8.2, C9.2, J3.1 (Pin_1), J5.6 (Pin_6), JP1.1 (A), JP2.2 (B), JP3.1 (A), JP4.1 (A), Q1.2 (E), R15.2, R16.2, R3.1, SW1.3 (C), U1.7 (GND), U1.9 (GND), U2.2 (GND), U3.4 (GND), U4.2 (GND)
- new net LCD_CS: J5.3 (Pin_3), R22.1
- new net LCD_DC: J5.2 (Pin_2), R17.1
- new net LCD_RST: J5.1 (Pin_1), R23.1
- new net MISO: R19.1, U3.2 (DO(IO1))
- new net MOSI: J5.5 (Pin_5), R21.1, U3.5 (DI(IO0))
- new net SCLK: J5.4 (Pin_4), R18.1, U3.6 (CLK)
- new net VBUS: F1.2, Q2.1 (E1), Q3.3 (D), U4.1 (5V)
- new net WS25_CS: R20.1, U3.1 (~{CS})
- no-connect marks 0 -> 1
Other:
- note added: "Charge current OPEN: 500mA SHORT: 1A"
- note added: "Display (4x M2.5)"
- note added: "IMPORTANT! Remove 3.3V LDO from ESP32-C3-ZERO board"
- note added: "Keypad (4x M2)"
- note added: "PCB (4x M2.5)"
- title: (none) -> CHIP-8 Portable

Commit message: chip8-pcb: final v2 version
Parts:
- removed H1, H2, H3, H4: ~, MountingHole:MountingHole_2.7mm_M2.5, symbol Mechanical:MountingHole
- removed H5, H6, H7, H8: ~, MountingHole:MountingHole_2.2mm_M2, symbol Mechanical:MountingHole
- H10, H11, H12, H9: footprint MountingHole:MountingHole_2.7mm_M2.5 -> MountingHole:MountingHole_2.2mm_M2
- J4: footprint chip8-pcb:AZDelivery_Keypad_4x4_Matrix_P2.54mm -> Connector_PinSocket_2.54mm:PinSocket_1x10_P2.54mm_Horizontal
Other:
- note added: "PCB (3x M2.5)"
- note removed: "Display (4x M2.5)"
- note removed: "Keypad (4x M2)"
- note removed: "PCB (4x M2.5)"
- moved on the sheet: BZ1, H10, H11, H12, J4, Q1, R10, R11, R12, R13, R14, R17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

Commit message: pcb: move battery and display connectors
Parts:
- J4: footprint Connector_PinSocket_2.54mm:PinSocket_1x10_P2.54mm_Horizontal -> Connector_PinSocket_2.54mm:PinSocket_1x08_P2.54mm_Horizontal
Connections:
- net at R7.2: now also J4.4 (R4); no longer J4.5 (R4)
- net at R11.2: now also J4.8 (C4); no longer J4.9 (C4)
- net at R4.2: now also J4.2 (R2); no longer J4.3 (R2)
- net at J4.1 (R1): now also R5.2
- net at R6.2: now also J4.3 (R3); no longer J4.4 (R3)
- net at R8.2: now also J4.5 (C1); no longer J4.6 (C1)
- net at R9.2: now also J4.6 (C2); no longer J4.7 (C2)
- net at R10.2: now also J4.7 (C3); no longer J4.8 (C3)
Changed lines of the file:
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@@
 			)
 		)
-		(property "Footprint" "Connector_PinSocket_2.54mm:PinSocket_1x10_P2.54mm_Horizontal"
+		(property "Footprint" "Connector_PinSocket_2.54mm:PinSocket_1x08_P2.54mm_Horizontal"
 			(at 116.84 115.57 0)
 			(effects
@@
 		(pin "7"
 		)
-		(pin "10"
-		)
-		(pin "9"
-		)
 		(instances
